Commit message: c6 cmt3

File: CHAPT6/chapt6_ws/src/fishbot_description/urdf/fishbot/actuator/caster.urdf.xacro (robot description, xacro)
@@ -1,13 +1,13 @@
 <?xml version="1.0"?>
 <robot xmlns:xacro="http://www.ros.org/wiki/xacro">
-    <xacro:macro name="camera_xacro" params="xyz">
-        <link name="camera_link">
+    <xacro:macro name="caster_xacro" params="caster_name xyz">
+        <link name="${caster_name}_link">
             <visual>
                 <origin xyz="0.0 0.0 0.0" rpy="0.0 0.0 0.0"/>
                 <geometry>
-                    <box size="0.02 0.10 0.02"/>
+                    <sphere radius="0.016"/>
                 </geometry>
-                <material name="black">
-                    <color rgba="0.0 0.0 0.0 0.5"/>
+                <material name="yellow">
+                    <color rgba="1.0 1.0 0.0 0.8"/>
                 </material>
             </visual>
@@ -15,15 +15,15 @@
                 <origin xyz="0.0 0.0 0.0" rpy="0.0 0.0 0.0"/>
                 <geometry>
-                    <box size="0.02 0.10 0.02"/>
+                    <sphere radius="0.016"/>
                 </geometry>
-                <material name="black">
-                    <color rgba="0.0 0.0 0.0 0.5"/>
+                <material name="yellow">
+                    <color rgba="1.0 1.0 0.0 0.8"/>
                 </material>
             </collision>
         </link>
-        <joint name="camera_joint" type="fixed">
+        <joint name="${caster_name}_joint" type="fixed">
             <origin xyz="${xyz}" rpy="0.0 0.0 0.0"/>
             <parent link="base_link"/>
-            <child link="camera_link"/>
+            <child link="${caster_name}_link"/>
         </joint>
     </xacro:macro>

File: CHAPT6/chapt6_ws/src/fishbot_description/urdf/fishbot/base.urdf.xacro (robot description, xacro)
@@ -1,5 +1,8 @@
 <?xml version="1.0"?>
 <robot xmlns:xacro="http://www.ros.org/wiki/xacro">
+    <xacro:include filename="$(find fishbot_description)/urdf/fishbot/common_inertial.xacro"/>
     <xacro:macro name="base_xacro" params="length radius">
+        <!--虚拟部件，贴地-->
+        <link name="base_footprint"/>
         <link name="base_link">
             <visual>
@@ -12,5 +15,20 @@
                 </material>
             </visual>
+            <collision>
+                <origin xyz="0.0 0.0 0.0" rpy="0.0 0.0 0.0"/>
+                <geometry>
+                    <cylinder radius="${radius}" length="${length}"/>
+                </geometry>
+                <material name="white">
+                    <color rgba="1.0 1.0 1.0 0.5"/>
+                </material>
+            </collision>
+            <xacro:cylinder_inertial m="1.0" r="${radius}" h="${length}"/>
         </link>
+        <joint name="joint_name" type="fixed">
+            <origin xyz="0.0 0.0 ${length/2.0+0.032-0.001}" rpy="0.0 0.0 0.0"/>
+            <parent link="base_footprint"/>
+            <child link="base_link"/>
+        </joint>
     </xacro:macro>
 </robot>

File: CHAPT6/chapt6_ws/src/fishbot_description/urdf/fishbot/fishrot.urdf.xacro (robot description, xacro)
@@ -1,11 +1,19 @@
 <?xml version="1.0"?>
 <robot xmlns:xacro="http://www.ros.org/wiki/xacro" name="fishbot">
-    <xacro:include filename="$(find fishbot_description)/urdf/fishbot/base.urdf.xacro"/>
-    <xacro:include filename="$(find fishbot_description)/urdf/fishbot/sensor/imu.urdf.xacro"/>
-    <xacro:include filename="$(find fishbot_description)/urdf/fishbot/sensor/camera.urdf.xacro"/>
-    <xacro:include filename="$(find fishbot_description)/urdf/fishbot/sensor/laser.urdf.xacro"/>
-    <xacro:base_xacro length="0.12" radius="0.10"/>
-    <xacro:imu_xacro xyz="0.0 0.0 0.02"/>
-    <xacro:camera_xacro xyz="0.10 0.0 0.075"/>
-    <xacro:laser_xacro xyz="0.0 0.0 0.10"/>
+  <!-- 包含子模块 -->
+  <xacro:include filename="$(find fishbot_description)/urdf/fishbot/base.urdf.xacro"/>
+  <xacro:include filename="$(find fishbot_description)/urdf/fishbot/sensor/imu.urdf.xacro"/>
+  <xacro:include filename="$(find fishbot_description)/urdf/fishbot/sensor/camera.urdf.xacro"/>
+  <xacro:include filename="$(find fishbot_description)/urdf/fishbot/sensor/laser.urdf.xacro"/>
+  <xacro:include filename="$(find fishbot_description)/urdf/fishbot/actuator/wheel.urdf.xacro"/>
+  <xacro:include filename="$(find fishbot_description)/urdf/fishbot/actuator/caster.urdf.xacro"/>
+  <!-- 实例化宏 -->
+  <xacro:base_xacro length="0.12" radius="0.10"/>
+  <xacro:imu_xacro xyz="0.0 0.0 0.02"/>
+  <xacro:camera_xacro xyz="0.10 0.0 0.075"/>
+  <xacro:laser_xacro xyz="0.0 0.0 0.10"/>
+  <xacro:wheel_xacro wheel_name="left_wheel" xyz="0.0 0.10 -0.06"/>
+  <xacro:wheel_xacro wheel_name="right_wheel" xyz="0.0 -0.10 -0.06"/>
+  <xacro:caster_xacro caster_name="front_caster" xyz="0.08 0.0 -0.076"/>
+  <xacro:caster_xacro caster_name="back_caster" xyz="-0.08 0.0 -0.076"/>
 </robot>

File: CHAPT6/chapt6_ws/src/fishbot_description/urdf/fishbot/sensor/imu.urdf.xacro (robot description, xacro)
@@ -12,4 +12,13 @@
                 </material>
             </visual>
+            <collision>
+                <origin xyz="0.0 0.0 0.0" rpy="0.0 0.0 0.0"/>
+                <geometry>
+                    <box size="0.02 0.02 0.02"/>
+                </geometry>
+                <material name="black">
+                    <color rgba="0.0 0.0 0.0 0.5"/>
+                </material>
+            </collision>
         </link>
         <joint name="imu_joint" type="fixed">

File: CHAPT6/chapt6_ws/src/fishbot_description/urdf/fishbot/sensor/laser.urdf.xacro (robot description, xacro)
@@ -12,4 +12,13 @@
                 </material>
             </visual>
+            <collision>
+                <origin xyz="0.0 0.0 0.0" rpy="0.0 0.0 0.0"/>
+                <geometry>
+                    <cylinder radius="0.01" length="0.10"/>
+                </geometry>
+                <material name="black">
+                    <color rgba="0.0 0.0 0.0 1.0"/>
+                </material>
+            </collision>
         </link>
         <link name="laser_link">
@@ -23,4 +32,13 @@
                 </material>
             </visual>
+            <collision>
+                <origin xyz="0.0 0.0 0.0" rpy="0.0 0.0 0.0"/>
+                <geometry>
+                    <cylinder radius="0.02" length="0.02"/>
+                </geometry>
+                <material name="black">
+                    <color rgba="0.0 0.0 0.0 0.5"/>
+                </material>
+            </collision>
         </link>
         <joint name="laser_joint" type="fixed">
